File: Hardware/BatterySwitchBoard_3S1P/BatterySwitchBoard_3S1P.brd (EAGLE design)
At the start: 88.9 x 53.1 mm, 31 parts, among them J1 5.5x2.1mm Barrel, Q1 DMG3404, U1 TPS22917DBV, U2 TPS22917DBV, U4 SN74AUP2G08DCU, U5 TLV3691DCK, U6 TPS56209, U7 MIC842L

Commit message: Added documentation and minor board updates
Parts:
- added VR1: POTENTIOMETER3214W, bschulz:POT_3214W
- R5: value 33.2k -> 4.7k
- moved R5 7.32 mm to (82.0, 6.60), turned to 90 degrees
- moved C1 1.02 mm to (83.3, 15.0)
- moved C2 1.02 mm to (81.2, 15.0)
- moved C3 1.02 mm to (77.3, 13.1)
- moved C4 1.02 mm to (77.3, 10.8)
- moved C5 1.02 mm to (80.0, 6.60)
- moved L1 1.02 mm to (78.6, 15.7)
- moved U6 1.02 mm to (77.3, 7.37)
- moved R4 0.92 mm to (76.6, 3.30), turned to 90 degrees
Connections:
- new net N$12: R5.1, VR1.1
- net N$8: now also VR1.2; no longer R5.1
Routing:
- net VDC: track 48.1 -> 38.2 mm
- net GND: track 138.7 -> 129.1 mm, vias 6 -> 12
- net N$12: track 0.00 -> 5.21 mm
- net N$8: track 4.15 -> 7.90 mm
- net VDC_HV: track 25.3 -> 26.3 mm
- added copper zone on layer 16, net GND
Other:
- board text added: "7.5 ~ 12V >250mA"
- board text added: "Project Killdeer 3S1P v1.0 Bobby Schulz"
- board text removed: "5 ~ 12V >250mA"
- board text removed: "Project Killdeer 3S1P v0.0 Bobby Schulz"
