File: Hardware/BatterySwitchBoard_3S1P/BatterySwitchBoard_3S1P.sch (EAGLE design)
At the start: 31 parts, among them J1 5.5x2.1mm Barrel, Q1 DMG3404, U1 TPS22917DBV, U2 TPS22917DBV, U4 SN74AUP2G08DCU, U5 TLV3691DCK, U6 TPS56209, U7 MIC842L

Commit message: Added documentation and minor board updates
Parts:
- added VR1: POTENTIOMETER3214W, bschulz:POTENTIOMETER3214W
- R5: value 33.2k -> 4.7k; device bschulz_passives:R-EU_33.2KR0603 -> bschulz_passives:R-EU_4.7KR0603
Connections:
- new net N$12: R5.1, VR1.A
- net N$8: now also VR1.S; no longer R5.1
Other:
- moved on the sheet: R4, R5
Changed lines of the file:
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@@
 <layer number="128" name="_bValues" color="7" fill="1" visible="no" active="yes"/>
 <layer number="129" name="Mask" color="7" fill="1" visible="no" active="yes"/>
+<layer number="130" name="SMDSTROOK" color="7" fill="1" visible="no" active="no"/>
 <layer number="131" name="tAdjust" color="7" fill="1" visible="no" active="yes"/>
 <layer number="132" name="bAdjust" color="7" fill="1" visible="no" active="yes"/>
+<layer number="133" name="bottom_silk" color="7" fill="1" visible="no" active="no"/>
+<layer number="134" name="mbFinish" color="7" fill="1" visible="no" active="no"/>
+<layer number="135" name="mtGlue" color="7" fill="1" visible="no" active="no"/>
+<layer number="136" name="mbGlue" color="7" fill="1" visible="no" active="no"/>
+<layer number="137" name="mtTest" color="7" fill="1" visible="no" active="no"/>
+<layer number="138" name="mbTest" color="7" fill="1" visible="no" active="no"/>
+<layer number="139" name="mtKeepout" color="7" fill="1" visible="no" active="no"/>
+<layer number="140" name="mbKeepout" color="7" fill="1" visible="no" active="no"/>
+<layer number="141" name="mtRestrict" color="7" fill="1" visible="no" active="no"/>
+<layer number="142" name="mbRestrict" color="7" fill="1" visible="no" active="no"/>
+<layer number="143" name="mvRestrict" color="7" fill="1" visible="no" active="no"/>
 <layer number="144" name="Drill_legend" color="7" fill="1" visible="no" active="yes"/>
+<layer number="145" name="mHoles" color="7" fill="1" visible="no" active="no"/>
+<layer number="146" name="mMilling" color="7" fill="1" visible="no" active="no"/>
+<layer number="147" name="mMeasures" color="7" fill="1" visible="no" active="no"/>
+<layer number="148" name="mDocument" color="7" fill="1" visible="no" active="no"/>
+<layer number="149" name="mReference" color="7" fill="1" visible="no" active="no"/>
 <layer number="150" name="Notes" color="7" fill="1" visible="no" active="yes"/>
 <layer number="151" name="HeatSink" color="7" fill="1" visible="no" active="yes"/>
@@
 <layer number="154" name="FabDoc2" color="7" fill="1" visible="no" active="yes"/>
 <layer number="155" name="FabDoc3" color="7" fill="1" visible="no" active="yes"/>
+<layer number="166" name="AntennaArea" color="7" fill="1" visible="no" active="no"/>
+<layer number="168" name="4mmHeightArea" color="7" fill="1" visible="no" active="no"/>
+<layer number="191" name="mNets" color="7" fill="1" visible="no" active="no"/>
+<layer number="192" name="mBusses" color="7" fill="1" visible="no" active="no"/>
+<layer number="193" name="mPins" color="7" fill="1" visible="no" active="no"/>
+<layer number="194" name="mSymbols" color="7" fill="1" visible="no" active="no"/>
+<layer number="195" name="mNames" color="7" fill="1" visible="no" active="no"/>
+<layer number="196" name="mValues" color="7" fill="1" visible="no" active="no"/>
 <layer number="199" name="Contour" color="7" fill="1" visible="no" active="yes"/>
 <layer number="200" name="200bmp" color="7" fill="1" visible="no" active="yes"/>
@@
 <part name="C5" library="bschulz_passives" deviceset="C-EU" device="C0603" technology="0.1UF" value="0.1uF"/>
 <part name="R4" library="bschulz_passives" deviceset="R-EU_" device="R0603" technology="10K" value="10k"/>
-<part name="R5" library="bschulz_passives" deviceset="R-EU_" device="R0603" technology="33.2K" value="33.2k"/>
 <part name="GND11" library="supply1" library_urn="urn:adsk.eagle:library:371" deviceset="GND" device=""/>
 <part name="GND12" library="supply1" library_urn="urn:adsk.eagle:library:371" deviceset="GND" device=""/>
@@
 <part name="BT3" library="bschulz" deviceset="AA" device="CLIP"/>
 <part name="H4" library="bschulz" deviceset="MOUNTING_HOLE" device="4_NP"/>
+<part name="VR1" library="bschulz" deviceset="POTENTIOMETER" device="3214W"/>
+<part name="R5" library="bschulz_passives" deviceset="R-EU_" device="R0603" technology="4.7K" value="4.7k"/>
 </parts>
 <sheets>
@@
 <attribute name="VALUE" x="118.364" y="107.061" size="1.778" layer="96"/>
 </instance>
-<instance part="R4" gate="G$1" x="134.62" y="99.06" smashed="yes" rot="R90">
-<attribute name="NAME" x="133.1214" y="95.25" size="1.778" layer="95" rot="R90"/>
-<attribute name="VALUE" x="137.922" y="95.25" size="1.778" layer="96" rot="R90"/>
-</instance>
-<instance part="R5" gate="G$1" x="134.62" y="109.22" smashed="yes" rot="R90">
-<attribute name="NAME" x="133.1214" y="105.41" size="1.778" layer="95" rot="R90"/>
-<attribute name="VALUE" x="137.922" y="105.41" size="1.778" layer="96" rot="R90"/>
-</instance>
-<instance part="GND11" gate="1" x="134.62" y="88.9" smashed="yes">
-<attribute name="VALUE" x="132.08" y="86.36" size="1.778" layer="96"/>
+<instance part="R4" gate="G$1" x="134.62" y="78.74" smashed="yes" rot="R90">
+<attribute name="NAME" x="133.1214" y="74.93" size="1.778" layer="95" rot="R90"/>
+<attribute name="VALUE" x="137.922" y="74.93" size="1.778" layer="96" rot="R90"/>
+</instance>
+<instance part="GND11" gate="1" x="134.62" y="68.58" smashed="yes">
+<attribute name="VALUE" x="132.08" y="66.04" size="1.778" layer="96"/>
 </instance>
 <instance part="GND12" gate="1" x="144.78" y="101.6" smashed="yes">
@@
 <attribute name="NAME" x="212.852" y="28.5242" size="1.778" layer="95"/>
 <attribute name="VALUE" x="212.852" y="25.4762" size="1.778" layer="96"/>
+</instance>
+<instance part="VR1" gate="G$1" x="139.7" y="91.44" smashed="yes" rot="R180">
+<attribute name="NAME" x="136.652" y="91.694" size="1.778" layer="95" font="vector" rot="R90"/>
+<attribute name="VALUE" x="140.97" y="91.44" size="1.778" layer="95" font="vector" rot="R270" align="bottom-center"/>
+</instance>
+<instance part="R5" gate="G$1" x="139.7" y="106.68" smashed="yes" rot="R90">
+<attribute name="NAME" x="138.2014" y="102.87" size="1.778" layer="95" rot="R90"/>
+<attribute name="VALUE" x="143.002" y="102.87" size="1.778" layer="96" rot="R90"/>
 </instance>
 </instances>
@@
 <segment>
 <pinref part="R4" gate="G$1" pin="1"/>
-<wire x1="134.62" y1="93.98" x2="134.62" y2="91.44" width="0.1524" layer="91"/>
+<wire x1="134.62" y1="73.66" x2="134.62" y2="71.12" width="0.1524" layer="91"/>
 <pinref part="GND11" gate="1" pin="GND"/>
 </segment>
@@
 <pinref part="L1" gate="G$1" pin="2"/>
 <pinref part="C1" gate="G$1" pin="1"/>
-<wire x1="132.08" y1="114.3" x2="134.62" y2="114.3" width="0.1524" layer="91"/>
 <pinref part="C2" gate="G$1" pin="1"/>
-<wire x1="134.62" y1="114.3" x2="144.78" y2="114.3" width="0.1524" layer="91"/>
+<wire x1="132.08" y1="114.3" x2="139.7" y2="114.3" width="0.1524" layer="91"/>
+<wire x1="139.7" y1="114.3" x2="144.78" y2="114.3" width="0.1524" layer="91"/>
 <wire x1="144.78" y1="114.3" x2="154.94" y2="114.3" width="0.1524" layer="91"/>
 <junction x="144.78" y="114.3"/>
@@
 <label x="162.56" y="114.3" size="1.778" layer="95" xref="yes"/>
 <pinref part="R5" gate="G$1" pin="2"/>
-<junction x="134.62" y="114.3"/>
+<wire x1="139.7" y1="111.76" x2="139.7" y2="114.3" width="0.1524" layer="91"/>
+<junction x="139.7" y="114.3"/>
 </segment>
 <segment>
@@
 <segment>
 <pinref part="R4" gate="G$1" pin="2"/>
-<pinref part="R5" gate="G$1" pin="1"/>
+<pinref part="VR1" gate="G$1" pin="S"/>
+<wire x1="134.62" y1="83.82" x2="134.62" y2="91.44" width="0.1524" layer="91"/>
 <pinref part="U6" gate="G$1" pin="VFB"/>
-<wire x1="134.62" y1="104.14" x2="114.3" y2="104.14" width="0.1524" layer="91"/>
-<junction x="134.62" y="104.14"/>
+<wire x1="114.3" y1="104.14" x2="127" y2="104.14" width="0.1524" layer="91"/>
+<wire x1="127" y1="104.14" x2="127" y2="91.44" width="0.1524" layer="91"/>
+<wire x1="127" y1="91.44" x2="134.62" y2="91.44" width="0.1524" layer="91"/>
+<junction x="134.62" y="91.44"/>
 </segment>
 </net>
@@
 </segment>
 </net>
+<net name="N$12" class="0">
+<segment>
+<pinref part="VR1" gate="G$1" pin="A"/>
+<pinref part="R5" gate="G$1" pin="1"/>
+<wire x1="139.7" y1="99.06" x2="139.7" y2="101.6" width="0.1524" layer="91"/>
+</segment>
+</net>
